File: H_Bridge/H_Bridge.kicad_sch (KiCad schematic)
At the start: 1 part, among them Q1 AO4614B

Commit message: new
Parts:
- added C1, C2: C, symbol EESTN5:C
- added Q2: AO4614B, symbol Mosfet:AO4614B
- added R1, R2: R, symbol EESTN5:R
- added U1, U2, U3: CD4093B, symbol Logic_Gate:CD4093B
Connections:
- net GND: now reaches Q1.1 (S)
- net GND: now also C1.2, C2.2, Q2.1 (S)
- net S2: now reaches Q1.2 (G)
- net S2: now also U3.4 (K)
- net OUT1: now reaches Q1.5 (D), Q1.6 (D), Q1.7 (D), Q1.8 (D)
- net VCC: now reaches Q1.3 (S)
- net VCC: now also Q2.3 (S)
- net S3: now reaches Q1.4 (G)
- net S3: now also U2.3 (J)
- new net: C2.1, R2.2, U3.2 (B)
- new net: U3.3 (J), U3.5 (C), U3.6 (D)
- new net: U2.1 (A), U2.4 (K)
- new net: R1.1, U1.3 (J), U2.5 (C), U2.6 (D)
- new net: U2.10 (L), U2.2 (B)
- new net: C1.1, R1.2, U2.8 (E), U2.9 (F)
- new net: U1.10 (L), U1.12 (G)
- new net: U1.1 (A), U1.4 (K)
- new net A0: Q2.2 (G), U1.2 (B), U1.8 (E), U1.9 (F)
- new net A1: R2.1, U1.13 (H), U1.5 (C), U1.6 (D), U3.1 (A)
- new net OUT2: Q2.5 (D), Q2.6 (D), Q2.7 (D), Q2.8 (D)
- new net S1: Q2.4 (G), U1.11 (M)
Other:
- moved on the sheet: Q1A, Q1B
