File: Sensors/Sensors.kicad_sch (KiCad schematic)
At the start: 19 parts, among them IC1 CD4051B, J2 Conn_01x06, Q1 TCRT5000, Q2 TCRT5000, Q3 TCRT5000, Q4 TCRT5000, Q5 TCRT5000, Q6 TCRT5000, Q7 TCRT5000, Q8 TCRT5000

Commit message: Rev. 1.0.0
Parts:
- removed IC1: CD4051B, MacroLib:DIP-16, symbol Logic_Gate:CD4051B
- removed J2: Conn_01x06, MacroLib:Pin_Header_Wire_6, symbol EESTN5:Conn_01x06
- added J1: CONN_01X10, MacroLib:Pin_Header_Wire_10, symbol MacroLib:CONN_01X10
- added J2, J3: Cable_PAD, EESTN5:Tornillo_M3_8mm, symbol EESTN5:Cable_PAD
- added R10, R11, R12, R2, R3, R5, R9: R, MacroLib:RES0.3, symbol EESTN5:R
- R1: value 10k -> R
Connections:
- net COM is gone; now on net CH_0: R1.1
- net CH_0: now also J1.9
- net CH_1: now also J1.8, R2.1
- net CH_2: now also J1.7, R3.1
- net CH_3: now also J1.6, R5.1
- net CH_4: now also J1.5, R9.1
- net CH_5: now also J1.4, R10.1
- net CH_6: now also J1.3, R11.1
- net CH_7: now also J1.2, R12.1
- net GND: now also J1.10, R10.2, R11.2, R12.2, R2.2, R3.2, R5.2, R9.2
- net VCC: now also J1.1
