File: Body/Body.kicad_pcb (KiCad board)
At the start: 2 copper layers, 127 x 100 mm, 30 parts, among them J1 Arduino_Nano_Header, J2 TB_1X2, J3 Cable_PAD, J4 TB_1X2, J5 TB_1X2, J6 Cable_PAD, J7 CONN_01X10, SW1 SW_SPDT, SW4 SW_Push, SW5 SW_Push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

Commit message: rev_0.0.1
Parts:
- removed R11: R, MacroLib:RES0.3
- added U3: DRV8833_MODULE, MacroLib:DRV8833_MODULE, F.Cu at (146.5, 99.0)
- moved R12 119.7 mm to (175.1, 142.7)
- moved SW4 116.7 mm to (175.1, 135.5), turned to 90 degrees
- moved U2 72.9 mm to (179.5, 116.3), turned to 90 degrees
- moved C4 70.4 mm to (168.1, 124.4)
- moved C1 68.8 mm to (168.4, 114.7), turned to 180 degrees
- moved C3 68.6 mm to (173.6, 124.4), turned to 90 degrees
- moved R6 68.0 mm to (150.9, 123.7)
- moved C2 64.4 mm to (173.6, 114.7), turned to -90 degrees
- moved R7 60.5 mm to (159.5, 103.0)
- moved R8 60.1 mm to (156.0, 103.0), turned to 90 degrees
- moved U1 53.8 mm to (129.5, 99.0)
- moved LED3 47.2 mm to (100.0, 122.2), turned to -90 degrees
- moved SW1 46.5 mm to (176.0, 95.7), turned to 90 degrees
- moved LED1 46.2 mm to (99.8, 101.4), turned to 90 degrees
- moved J2 44.1 mm to (174.9, 104.5), turned to 0 degrees
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Connections:
- net Net-(U1-OUT1) renamed /OUT1
- net Net-(U1-OUT2) renamed /OUT2
- net Net-(U1-OUT3) renamed /OUT3
- net Net-(U1-OUT4) renamed /OUT4
- C1 pad 1: VCC -> +7.5V
- C2 pad 1: VCC -> +7.5V
- J1 pad 30: VCC -> +7.5V
- J1 pad 8: Net-(J1-D5/T1) -> unconnected-(J1-D5/T1-Pad8)
- J2 pad 1: Net-(SW1-A) -> VCC
- LED1 pad 1: VCC -> Net-(LED1-A)
- LED1 pad 2: Net-(LED1-K) -> GND
- R1 pad 1: Net-(LED1-K) -> +7.5V
- R1 pad 2: GND -> Net-(LED1-A)
- R7 pad 1: /IN1A -> /IN2A
- R8 pad 2: /IN2A -> /IN1A
- SW1 pad 1: Net-(SW1-A) -> VCC
- SW1 pad 2: VCC -> +7.5V
- U1 pad 12: /EN -> unconnected-(U1-EPP-Pad12)
- U2 pad 3: VCC -> +7.5V
Routing:
- net /ULT: track 0.00 -> 79.3 mm, vias 0 -> 2
- net /OUT1: track 0.00 -> 77.5 mm
- net /OUT2: track 0.00 -> 70.7 mm
- net /OUT3: track 0.00 -> 66.1 mm
- net /OUT4: track 0.00 -> 58.2 mm
- net /IN2B: track 0.00 -> 54.1 mm
- net /IN1B: track 0.00 -> 47.0 mm
- net /IN2A: track 0.00 -> 35.0 mm
- net Net-(J1-D9/0C1): track 0.00 -> 33.5 mm
- net /IN1A: track 0.00 -> 25.6 mm
- net Net-(J1-D3/INT1): track 0.00 -> 21.6 mm
- net Net-(J1-D11/MOSI): track 0.00 -> 17.8 mm
- net Net-(J1-D10/SS): track 0.00 -> 17.0 mm
- net /S5: track 0.00 -> 9.60 mm
- net /S4: track 0.00 -> 9.55 mm
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- added copper zone on B.Cu, net GND
Other:
- board size 127 x 100 mm -> 100 x 99.5 mm

Commit message: new
Parts:
- moved R1 67.5 mm to (167.2, 91.8)
- moved R4 31.6 mm to (117.5, 132.8)
- moved R5 26.0 mm to (117.5, 136.0)
- moved R7 22.2 mm to (143.1, 118.0)
- moved R8 22.2 mm to (139.6, 118.0)
- moved R10 18.5 mm to (122.6, 118.0)
- moved R9 18.5 mm to (125.6, 118.0)
- moved R13 17.3 mm to (117.5, 139.2)
- moved R6 15.1 mm to (161.5, 134.5)
- moved R12 14.2 mm to (161.5, 138.5)
- moved J7 12.2 mm to (136.7, 154.0)
- moved J1 10.8 mm to (138.0, 136.0)
- moved J2 8.24 mm to (167.5, 100.9), turned to 90 degrees
- moved LED1 7.61 mm to (106.5, 97.8), turned to -90 degrees
- moved U2 7.34 mm to (179.0, 123.6)
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Connections:
- J1 pad 10: /OUT_LED2 -> /OUT_LED1
- J1 pad 9: /OUT_LED1 -> /OUT_LED2
- LED2 pad 1: /OUT_LED1 -> Net-(LED2-A)
- LED2 pad 2: Net-(LED2-K) -> GND
- LED3 pad 1: /OUT_LED2 -> Net-(LED3-A)
- LED3 pad 2: Net-(LED3-K) -> GND
- R4 pad 1: Net-(LED2-K) -> /OUT_LED1
- R4 pad 2: GND -> Net-(LED2-A)
- R5 pad 1: Net-(LED3-K) -> /OUT_LED2
- R5 pad 2: GND -> Net-(LED3-A)
Routing:
- net +5V: track 0.00 -> 66.0 mm
- net Net-(LED1-A): track 0.00 -> 64.4 mm
- net +7.5V: track 0.00 -> 49.7 mm
- net VCC: track 9.25 -> 57.4 mm
- net /IN_BUTTON1: track 0.00 -> 25.1 mm
- net Net-(LED2-A): track 0.00 -> 25.0 mm
- net Net-(J1-D9/0C1): track 33.5 -> 16.0 mm
- net Net-(J1-D3/INT1): track 21.6 -> 5.31 mm
- net /IN1A: track 25.6 -> 9.59 mm
- net Net-(LED3-A): track 0.00 -> 14.7 mm
- net Net-(J1-D11/MOSI): track 17.8 -> 5.37 mm
- net /IN2A: track 35.0 -> 23.2 mm
- net Net-(J1-D10/SS): track 17.0 -> 5.43 mm
- net /IN1B: track 47.0 -> 41.8 mm
- net /ULT: track 79.3 -> 84.6 mm
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Other:
- board size 100 x 99.5 mm -> 100 x 115.5 mm

Commit message: new
Parts:
- moved U2 9.59 mm to (170.2, 119.7), turned to 0 degrees
- moved C3 2.45 mm to (173.0, 129.0)
- moved C4 1.99 mm to (166.8, 128.7)
- moved J7 1.22 mm to (137.9, 154.0)
- moved C1 0.50 mm to (167.3, 111.6), turned to 0 degrees
- moved SW4 0.50 mm to (174.0, 139.0)
- moved C2 0.10 mm to (173.0, 111.5), turned to 90 degrees
Routing:
- net +7.5V: track 49.7 -> 108.1 mm
- net /OUT_LED2: track 0.00 -> 19.8 mm
- net /OUT1: track 78.4 -> 96.8 mm
- net /IN_BUTTON2: track 0.00 -> 16.2 mm
- net /OUT_LED1: track 0.00 -> 13.8 mm
- net /IN_BUTTON1: track 25.1 -> 38.5 mm
- net +5V: track 66.0 -> 52.7 mm
- net Net-(R13-Pad1): track 0.00 -> 11.4 mm
- net Net-(R12-Pad1): track 0.00 -> 8.68 mm
- net /IN1B: track 41.8 -> 48.8 mm
- net /OUT4: track 61.9 -> 59.6 mm
- net /OUT3: track 69.0 -> 67.9 mm
- net /IN2B: track 50.6 -> 51.3 mm
- net /S5: track 10.4 -> 10.9 mm
- net /S2: track 10.4 -> 10.9 mm
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Other:
- board size 100 x 115.5 mm -> 94 x 115.5 mm

Commit message: Rev. 1.0.0
Parts:
- added J8: Cable_PAD, EESTN5:Tornillo_M3_8mm, F.Cu at (119.0, 158.0)
- added J9: Cable_PAD, EESTN5:Tornillo_M3_8mm, F.Cu at (157.0, 158.0)
Other:
- outline, holes or cut-outs redrawn

Commit message: V1.0.0
Parts:
- added G***: LOGO, EESTN5:LOGO_Cu, B.Cu at (113.0, 149.0)
- moved C3 2.06 mm to (172.5, 127.0)
Routing:
- net +5V: track 52.7 -> 51.5 mm
Other:
- board text added: "BOTT1"
- board text added: "BOTT2"
- board text added: "POWER"
- board text added: "SYS1"
- board text added: "SYS2"

Commit message: Rev 1.0.1
Parts:
- U2: value LM78XX -> L7805
- moved U2 1.70 mm to (170.2, 118.0), turned to 180 degrees
Connections:
- J7 pad 1: +5V -> GND
- J7 pad 10: GND -> +5V
- U2 pad 1: GND -> +7.5V
- U2 pad 2: +5V -> GND
- U2 pad 3: +7.5V -> +5V
Routing:
- net +5V: track 51.5 -> 85.2 mm, vias 0 -> 2
- net +7.5V: track 108.1 -> 99.9 mm
