File: Body/Body.kicad_sch (KiCad schematic)
At the start: 30 parts, among them J1 Arduino_Nano_Header, J2 TB_1X2, J3 Cable_PAD, J4 TB_1X2, J5 TB_1X2, J6 Cable_PAD, J7 CONN_01X10, SW1 SW_SPDT, SW4 SW_Push, SW5 SW_Push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

Commit message: rev_0.0.1
Parts:
- removed R11: R, MacroLib:RES0.3, symbol EESTN5:R
- added U3: DRV8833_MODULE, MacroLib:DRV8833_MODULE, symbol MacroLib:DRV8833_MODULE
Connections:
- net GND: now also LED1.2 (K), U3.3 (GND); no longer R1.2
- net IN1A: now also R8.2, U3.1 (IN4); no longer R7.1
- net IN1B: now also U3.5 (IN2)
- net IN2A: now also R7.1, U3.2 (IN3); no longer R8.2
- net IN2B: now also U3.6 (IN1)
- net ULT: now also U3.7 (ULT)
- net VCC: now also J2.1, SW1.1 (A), U3.4 (VCC); no longer C1.1, C2.1, J1.30 (VIN), LED1.1 (A), SW1.2 (B), U2.3 (VIN)
- net +7.5V: now reaches R1.1
- net +7.5V: now also C1.1, C2.1, J1.30 (VIN), SW1.2 (B), U2.3 (VIN); no longer LED1.2 (K)
- net OUT2: now reaches J5.1, U1.10 (OUT2)
- net OUT2: now also U3.9 (OUT3)
- net OUT1: now reaches J5.2, U1.11 (OUT1)
- net OUT1: now also U3.8 (OUT4)
- net OUT4: now reaches J4.1, U1.8 (OUT4)
- net OUT4: now also U3.11 (OUT1)
- net OUT3: now reaches J4.2, U1.9 (OUT3)
- net OUT3: now also U3.10 (OUT2)
- net EN: no longer names the net of U1.12 (EPP)
- new net: LED1.1 (A), R1.2
Other:
- moved on the sheet: C1, C2, C3, C4, J4, J5, LED1, R1, R6, U1, U2

Commit message: new
Connections:
- net GND: now also LED2.2 (K), LED3.2 (K); no longer R4.2, R5.2
- net OUT_LED1: now also J1.10 (D7/AIN1), R4.1; no longer J1.9 (D6/AIN0), LED2.1 (A)
- net OUT_LED2: now also J1.9 (D6/AIN0), R5.1; no longer J1.10 (D7/AIN1), LED3.1 (A)
- new net: LED2.1 (A), R4.2
- new net: LED3.1 (A), R5.2
Other:
- moved on the sheet: LED2, LED3, R4, R5
Changed lines of the file:
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@@
 	(wire
 		(pts
-			(xy 125.73 160.02) (xy 125.73 163.83)
+			(xy 125.73 161.29) (xy 125.73 165.1)
 		)
 		(stroke
@@
 	(wire
 		(pts
-			(xy 106.68 160.02) (xy 106.68 163.83)
+			(xy 106.68 161.29) (xy 106.68 165.1)
 		)
 		(stroke
@@
 	)
 	(label "OUT_LED2"
-		(at 154.94 125.73 180)
+		(at 154.94 123.19 180)
 		(fields_autoplaced yes)
 		(effects
@@
 	)
 	(label "OUT_LED1"
-		(at 154.94 123.19 180)
+		(at 154.94 125.73 180)
 		(fields_autoplaced yes)
 		(effects
@@
 	(symbol
 		(lib_id "EESTN5:R")
-		(at 106.68 166.37 0)
+		(at 106.68 158.75 0)
 		(unit 1)
 		(exclude_from_sim no)
@@
 		(fields_autoplaced yes)
 		(property "Reference" "R4"
-			(at 107.95 165.0999 0)
+			(at 107.95 157.4799 0)
 			(effects
 				(font
@@
 		)
 		(property "Value" "R"
-			(at 107.95 167.6399 0)
+			(at 107.95 160.0199 0)
 			(effects
 				(font
@@
 		)
 		(property "Footprint" "MacroLib:RES0.3"
-			(at 106.68 166.37 0)
+			(at 106.68 158.75 0)
 			(effects
 				(font
@@
 		)
 		(property "Datasheet" ""
-			(at 106.68 166.37 0)
+			(at 106.68 158.75 0)
 			(effects
 				(font
@@
 		)
 		(property "Description" "Resistor"
-			(at 106.68 166.37 0)
+			(at 106.68 158.75 0)
 			(effects
 				(font
@@
 	(symbol
 		(lib_id "EESTN5:R")
-		(at 125.73 166.37 0)
+		(at 125.73 158.75 0)
 		(unit 1)
 		(exclude_from_sim no)
@@
 		(fields_autoplaced yes)
 		(property "Reference" "R5"
-			(at 127 165.0999 0)
+			(at 127 157.4799 0)
 			(effects
 				(font
@@
 		)
 		(property "Value" "R"
-			(at 127 167.6399 0)
+			(at 127 160.0199 0)
 			(effects
 				(font
@@
 		)
 		(property "Footprint" "MacroLib:RES0.3"
-			(at 125.73 166.37 0)
+			(at 125.73 158.75 0)
 			(effects
 				(font
@@
 		)
 		(property "Datasheet" ""
-			(at 125.73 166.37 0)
+			(at 125.73 158.75 0)
 			(effects
 				(font
@@
 		)
 		(property "Description" "Resistor"
-			(at 125.73 166.37 0)
+			(at 125.73 158.75 0)
 			(effects
 				(font
@@
 	(symbol
 		(lib_id "EESTN5:LED")
-		(at 125.73 157.48 270)
+		(at 125.73 166.37 270)
 		(unit 1)
 		(exclude_from_sim no)
@@
 		(fields_autoplaced yes)
 		(property "Reference" "LED3"
-			(at 127 156.9719 90)
+			(at 127 165.8619 90)
 			(effects
 				(font
@@
 		)
 		(property "Value" "LED"
-			(at 127 159.5119 90)
+			(at 127 168.4019 90)
 			(effects
 				(font
@@
 		)
 		(property "Footprint" "EESTN5:led_5mm_green"
-			(at 125.73 157.48 0)
+			(at 125.73 166.37 0)
 			(effects
 				(font
@@
 		)
 		(property "Datasheet" ""
-			(at 125.73 157.48 0)
+			(at 125.73 166.37 0)
 			(effects
 				(font
@@
 		)
 		(property "Description" ""
-			(at 125.73 157.48 0)
+			(at 125.73 166.37 0)
 			(effects
 				(font
@@
 	(symbol
 		(lib_id "EESTN5:LED")
-		(at 106.68 157.48 270)
+		(at 106.68 166.37 270)
 		(unit 1)
 		(exclude_from_sim no)
@@
 		(fields_autoplaced yes)
 		(property "Reference" "LED2"
-			(at 107.95 156.9719 90)
+			(at 107.95 165.8619 90)
 			(effects
 				(font
@@
 		)
 		(property "Value" "LED"
-			(at 107.95 159.5119 90)
+			(at 107.95 168.4019 90)
 			(effects
 				(font
@@
 		)
 		(property "Footprint" "EESTN5:led_5mm_green"
-			(at 106.68 157.48 0)
+			(at 106.68 166.37 0)
 			(effects
 				(font
@@
 		)
 		(property "Datasheet" ""
-			(at 106.68 157.48 0)
+			(at 106.68 166.37 0)
 			(effects
 				(font
@@
 		)
 		(property "Description" ""
-			(at 106.68 157.48 0)
+			(at 106.68 166.37 0)
 			(effects
 				(font

Commit message: Rev. 1.0.0
Parts:
- added J8, J9: Cable_PAD, EESTN5:Tornillo_M3_8mm, symbol EESTN5:Cable_PAD
Changed lines of the file:
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@@
+	)
+	(symbol
+		(lib_id "EESTN5:Cable_PAD")
+		(at 147.32 60.96 0)
+		(unit 1)
+		(exclude_from_sim no)
+		(in_bom yes)
+		(on_board yes)
+		(dnp no)
+		(fields_autoplaced yes)
+		(property "Reference" "J9"
+			(at 149.86 60.9599 0)
+			(effects
+				(font
+					(size 1.27 1.27)
+				)
+				(justify left)
+			)
+		)
+		(property "Value" "Cable_PAD"
+			(at 147.32 57.785 0)
+			(effects
+				(font
+					(size 1.27 1.27)
+				)
+				(hide yes)
+			)
+		)
+		(property "Footprint" "EESTN5:Tornillo_M3_8mm"
+			(at 147.32 60.96 0)
+			(effects
+				(font
+					(size 1.524 1.524)
+				)
+				(hide yes)
+			)
+		)
+		(property "Datasheet" ""
+			(at 147.32 60.96 0)
+			(effects
+				(font
+					(size 1.524 1.524)
+				)
+				(hide yes)
+			)
+		)
+		(property "Description" "Solder Pad for cable connection"
+			(at 147.32 60.96 0)
+			(effects
+				(font
+					(size 1.27 1.27)
+				)
+				(hide yes)
+			)
+		)
+		(pin "1"
+		)
+		(instances
+			(project "Body"
+				(path "/6c5b21d1-f71a-47c4-bb84-a535bf65c72e"
+					(reference "J9")
+					(unit 1)
+				)
+			)
+		)
 	)
 	(symbol
@@
 					(unit 1)
 				)
+			)
+		)
+	)
+	(symbol
+		(lib_id "EESTN5:Cable_PAD")
+		(at 147.32 53.34 0)
+		(unit 1)
+		(exclude_from_sim no)
+		(in_bom yes)
+		(on_board yes)
+		(dnp no)
+		(fields_autoplaced yes)
+		(property "Reference" "J8"
+			(at 149.86 53.3399 0)
+			(effects
+				(font
+					(size 1.27 1.27)
+				)
+				(justify left)
+			)
+		)
+		(property "Value" "Cable_PAD"
+			(at 147.32 50.165 0)
+			(effects
+				(font
+					(size 1.27 1.27)
+				)
+				(hide yes)
+			)
+		)
+		(property "Footprint" "EESTN5:Tornillo_M3_8mm"
+			(at 147.32 53.34 0)
+			(effects
+				(font
+					(size 1.524 1.524)
+				)
+				(hide yes)
+			)
+		)
+		(property "Datasheet" ""
+			(at 147.32 53.34 0)
+			(effects
+				(font
+					(size 1.524 1.524)
+				)
+				(hide yes)
+			)
+		)
+		(property "Description" "Solder Pad for cable connection"
+			(at 147.32 53.34 0)
+			(effects
+				(font
+					(size 1.27 1.27)
+				)
+				(hide yes)
+			)
+		)
+		(pin "1"
+		)
+		(instances
+			(project "Body"
+				(path "/6c5b21d1-f71a-47c4-bb84-a535bf65c72e"
+					(reference "J8")
+					(unit 1)
+				)

Commit message: Rev 1.0.1
Parts:
- removed U2: LM78XX, MacroLib:TO-220-3_Vertical, symbol MacroLib:LM78XX
- added U2: L7805, MacroLib:TO-220-3_Vertical, symbol Regulator_Linear:L7805
Connections:
- net +5V: now also J7.10, U2.3 (OUT); no longer J7.1
- net +7.5V: now also U2.1 (IN)
- net GND: now also J7.1, U2.2 (GND); no longer J7.10
Other:
- moved on the sheet: C1, C2, C3, C4, J1, J2, J3, J4, J5, J6, J7, J8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
