File: ILARDOX/H BRIDGE.kicad_sch (KiCad schematic)
At the start: 44 parts, among them Q1 AO4614B, Q10 MMBT2222A, Q11 MMBT2907A, Q12 AO4614B, Q13 MMBT2222A, Q14 MMBT2222A, Q15 MMBT2907A, Q16 AO4614B, Q2 MMBT2222A, Q3 MMBT2907A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

Commit message: new
Parts:
- added C14, C15, C16, C17, C18, C19: C, symbol Device:C
Connections:
- net +BATT: now also C14.1, C15.1, C16.1, C17.1, C18.1, C19.1
- net GND: now also C14.2, C15.2, C16.2, C17.2, C18.2, C19.2
